Commit message: pnly the package, trial data and reconstruction

File: src/control/urdf/r1_rover.urdf (robot description, URDF)
Before this commit: robot r1_rover, 10 links, 9 joints
Links:
- link base_link: geometry visual mesh filename=package://control/urdf/meshes/chassis_link.STL scale=1 1 1
- link battery_link: geometry visual mesh filename=package://control/urdf/meshes/battery_link.STL scale=1 1 1
- link housing_link: geometry visual mesh filename=package://control/urdf/meshes/housing_link.STL scale=1 1 1
- link l_antenna_link: geometry visual mesh filename=package://control/urdf/meshes/antenna_link.STL scale=1 1 1
- link lb_wheel_link: geometry visual mesh filename=package://control/urdf/meshes/wheel_link.STL scale=1 1 1
- link lf_wheel_link: geometry visual mesh filename=package://control/urdf/meshes/wheel_link.STL scale=1 1 1
- link r_antenna_link: geometry visual mesh filename=package://control/urdf/meshes/antenna_link.STL scale=1 1 1
- link rb_wheel_link: geometry visual mesh filename=package://control/urdf/meshes/wheel_link.STL scale=1 1 1
- link rf_wheel_link: geometry visual mesh filename=package://control/urdf/meshes/wheel_link.STL scale=1 1 1
- link top_link: geometry visual mesh filename=package://control/urdf/meshes/top_link.STL scale=1 1 1
